Commit message: fixed mid points in URDF, put txt files in data folder

File: data/tensegrity_wrongMid/robots/tensegrity.URDF (robot description, URDF)
Before this commit: robot tensegrity, 52 links, 51 joints
Links:
- link pulley7: mass 0.00115149136839392 -> 0.00115149136839393
- link pulley9: mass 0.00115149136839395 -> 0.00115149136839394
- link tendon2: mass 0.0111536592298929 -> 0.0106761371465473
- link tightener2: mass 0.00856464520084458 -> 0.00856464520084457
- link tightener8: mass 0.00856465792468904 -> 0.00856465792468896
Joints:
- joint mid3: origin xyz=-0.0353270434653113 0.0203960780543712 1.288 rpy=-1.0471975511966 1.5707963267949 0 -> xyz=-0.0353270434653113 0.0203960780543712 1.288 rpy=1.0471975511966 1.5707963267949 0
- joint mid6: origin xyz=-0.0353270434653115 -0.0203960780543711 1.288 rpy=-2.0943951023932 1.5707963267949 0 -> xyz=-0.0353270434653115 -0.0203960780543711 1.288 rpy=2.0943951023932 1.5707963267949 0
- joint pulley1: axis 0 0 -1 -> 0 0 0
- joint pulley2: axis 0 0 -1 -> 0 0 0
- joint pulley3: axis 0 0 -1 -> 0 0 0
- joint pulley4: axis 0 0 -1 -> 0 0 0
- joint pulley5: axis 0 0 1 -> 0 0 0
- joint pulley6: axis 0 0 -1 -> 0 0 0
- joint pulley7: axis 0 0 -1 -> 0 0 0
- joint pulley8: axis 0 0 1 -> 0 0 0
- joint pulley9: axis 0 0 1 -> 0 0 0
