Commit message: return vector of inverse kinematic angles

File: data/tensegrity/robots/tensegrity.URDF (robot description, URDF)
Before this commit: robot tensegrity, 46 links, 45 joints
Links:
- link attach9: mass 0.000125397117258044 -> 0.000125397117258043
- link detach2: mass 0.00144131652160448 -> 0.00144131652160447
- link tendon1: mass 0.0112203866578552 -> 0.0103991743382068
- link tendon2: mass 0.0122147635645694 -> 0.0111099282601549
- link tendon3: mass 0.0118593866035953 -> 0.0109723265019277
- link tendon4: mass 0.0151436075636581 -> 0.0142485049847973
- link tendon5: mass 0.010344259298622 -> 0.00943206645572571
- link tendon6: mass 0.0128653245712748 -> 0.0117808467872556
- link tendon7: mass 0.00829493557883235 -> 0.0071673551436059
- link tendon8: mass 0.00996651419795441 -> 0.00906487710637413
- link tendon9: mass 0.0119694680101771 -> 0.0109763477405243
- link tensegrity: mass 3.0323 -> 2.981
- link tightener1: mass 0.0085646299641912 -> 0.00856462996419102
- link tightener2: mass 0.00856464520084467 -> 0.00856464520084429
- link tightener3: mass 0.00856463183459587 -> 0.00856463183459565
- link tightener4: mass 0.00856463280589166 -> 0.00856463280589177
- link tightener5: mass 0.00856464027785634 -> 0.00856464027785648
- link tightener6: mass 0.00856463401560633 -> 0.00856463401560627
- link tightener7: mass 0.00856463670998747 -> 0.00856463670998778
- link tightener8: mass 0.00856465792468872 -> 0.00856465792468896
- link tightener9: mass 0.00856463882730575 -> 0.00856463882730577
Joints:
- removed joint detach1
- added joint detach: type fixed, parent tensegrity, child detach1, origin xyz=0.0199999999999996 0.393098360655766 1.49733196721311 rpy=0 -0.181319774401501 -1.5707963267949, axis 0 0 0
- joint attach1: origin xyz=0.330836180337652 0.0959207585222343 1.96919528368496 rpy=-0.531711673196898 0.769136226420716 -2.96318215423882 -> xyz=0.318156761076164 0.0650930969857314 1.97852563931339 rpy=-0.531711673196898 0.769136226420716 -2.96318215423882
- joint attach2: origin xyz=-0.386688019933338 0.197454290583016 1.93990580280716 rpy=0.531711673196865 0.769136226420715 -0.178410499351044 -> xyz=-0.328656761076175 0.166626629046522 1.94923615843558 rpy=0.531711673196865 0.769136226420715 -0.178410499351044
- joint attach3: origin xyz=-0.659713818386888 -0.128493991794642 1.09364244438357 rpy=-2.6098809803929 -0.769136226420708 0.178410499351032 -> xyz=-0.601682559529722 -0.146570547440898 1.17252428668608 rpy=-2.6098809803929 -0.769136226420708 0.178410499351032
- joint attach4: origin xyz=0.559420853294264 -0.0203686209826116 1.0179626488128 rpy=1.03908465359801 -0.769136226420713 2.96318215423876 -> xyz=0.546741434032771 -0.0384451766288569 1.09684449111531 rpy=1.03908465359801 -0.769136226420713 2.96318215423876
- joint attach5: origin xyz=0.00132408020216285 -0.619952126384783 1.66259807389183 rpy=-2.35619449019234 0.181319774401488 1.57079632679489 -> xyz=0.0239999999999999 -0.59522390710731 1.69768777941467 rpy=-2.35619449019234 0.181319774401499 1.5707963267949
- joint attach6: origin xyz=0.603861978791218 -0.0269604597338994 1.06435296350577 rpy=2.60988098039293 -0.769136226420717 2.96318215423874 -> xyz=0.591182559529726 -0.0450370153801445 1.14323480580828 rpy=2.60988098039293 -0.769136226420713 2.96318215423875
- joint attach7: origin xyz=-0.386688019933338 0.197454290583016 1.93990580280716 rpy=-2.10250799999181 0.769136226420727 -2.96318215423883 -> xyz=0.273715635579209 0.0585012582344451 2.02491595400636 rpy=-2.10250799999181 0.769136226420727 -2.96318215423883
- joint attach8: origin xyz=-0.0466759197978372 0.696113447385709 1.42131938536724 rpy=-2.35619449019234 -0.181319774401499 -1.5707963267949 -> xyz=-0.0240000000000005 0.622481010925478 1.47444187777533 rpy=-2.35619449019234 -0.181319774401499 -1.5707963267949
- joint attach9: origin xyz=0.00132408020216294 0.682102245206886 1.34489464621002 rpy=0.785398163397449 -0.181319774401489 -1.57079632679489 -> xyz=0.0239999999999996 0.608469808746655 1.39801713861811 rpy=0.785398163397449 -0.181319774401489 -1.57079632679489
- joint detach2: origin xyz=-0.421921414642284 -0.075053824261462 1.26479790365546 rpy=1.31710983659433 -0.769136226420714 0.178410499351039 -> xyz=-0.421300155349653 -0.0844233171255465 1.31741827022436 rpy=1.31710983659433 -0.769136226420714 0.178410499351039
- joint detach3: origin xyz=-0.0336759197978377 -0.379170842228293 1.59929144201814 rpy=1.5707963267949 0.181319774401488 1.5707963267949 -> xyz=-0.0110000000000003 -0.366245901639344 1.63654508196721 rpy=1.5707963267949 0.181319774401488 1.5707963267949
- joint detach4: origin xyz=-0.377861591106548 -0.0785407278054665 1.34393297523359 rpy=1.31710983659433 -0.769136226420712 0.178410499351048 -> xyz=-0.32831561362362 -0.09814741615855 1.41446863913521 rpy=1.31710983659433 -0.769136226420712 0.178410499351048
- joint detach5: origin xyz=0.13726569898783 0.0143510786049931 1.85061555565431 rpy=0.253686490200554 0.769136226420712 -2.96318215423876 -> xyz=0.124586279726341 -0.0164765829315123 1.85994591128273 rpy=0.253686490200554 0.769136226420711 -2.96318215423876
- joint detach6: origin xyz=-0.00267591979783714 -0.249826579933211 1.57557832726404 rpy=1.5707963267949 0.181319774401488 1.5707963267949 -> xyz=0.0199999999999994 -0.236901639344262 1.61283196721312 rpy=1.5707963267949 0.181319774401488 1.5707963267949
- joint detach7: origin xyz=-0.0765515214055373 0.113257206654859 1.72464898138088 rpy=1.31710983659433 0.769136226420715 -0.178410499351034 -> xyz=-0.0270055439226141 0.0839596778251951 1.74232551541019 rpy=1.31710983659433 0.769136226420715 -0.178410499351034
- joint detach8: origin xyz=-0.16953606313157 0.160516714179241 1.81051902242288 rpy=1.31710983659433 0.769136226420716 -0.178410499351032 -> xyz=-0.119990085648646 0.131219185349568 1.82819555645219 rpy=1.31710983659433 0.769136226420715 -0.178410499351032
- joint detach9: origin xyz=0.438575768688868 0.0203654002444033 1.21796640096016 rpy=0.253686490200553 -0.769136226420708 2.96318215423877 -> xyz=0.425896349427369 0.00228884459815839 1.29684824326267 rpy=0.253686490200553 -0.769136226420708 2.96318215423877
- joint pulley1: origin xyz=-0.0466759197978372 0.696113447385709 1.42131938536724 rpy=1.5707963267949 -1.35303842246507 -1.5707963267949 -> xyz=0 0.621786885245901 1.47065573770492 rpy=1.5707963267949 -1.35303842246507 -1.5707963267949
- joint pulley2: origin xyz=-0.631486529546608 -0.0755513717494224 1.055238553721 rpy=0.631420863095884 0.532284485238217 -2.35588130681373 -> xyz=-0.573455270689443 -0.0936279273956821 1.13412039602351 rpy=0.631420863095884 0.532284485238217 -2.35588130681373
- joint pulley3: origin xyz=-0.0576759197978372 -0.627713495578133 1.62026333283719 rpy=2.98449472353879 -0.0909133937987542 -0.520440071048007 -> xyz=-0.0350000000000004 -0.60298527630066 1.65535303836004 rpy=2.98449472353879 -0.0909133937987541 -0.520440071048006
- joint pulley4: origin xyz=-0.654713818386888 -0.136350779806313 1.08999952218571 rpy=0.745639043009377 0.327890658213947 -2.08475010947139 -> xyz=-0.572811013144504 -0.162596564002146 1.14610965089734 rpy=0.745639043009377 0.327890658213947 -2.08475010947139
- joint pulley5: origin xyz=0.286395054840697 0.089328919770948 2.01558559837794 rpy=1.36772787967172 0.464271853741143 -0.0919392370595982 -> xyz=0.276437460986168 0.0428433090569649 2.02501938885851 rpy=1.36772787967172 0.464271853741143 -0.0919392370595983
- joint pulley6: origin xyz=-0.0576759197978372 -0.627713495578133 1.62026333283719 rpy=3.12170686669581 0.180237919378081 1.4603031742211 -> xyz=0.0349999999999996 -0.603075440235086 1.65486123508135 rpy=3.12170686669581 0.180237919378081 1.4603031742211
- joint pulley7: origin xyz=0.289116880247657 0.0736709705934651 2.01568903323008 rpy=2.37738677488523 -0.271358663823416 -1.66506917334562 -> xyz=-0.310210537417404 0.111920210362038 1.97801932924749 rpy=2.37738677488523 -0.271358663823417 -1.66506917334562
- joint pulley8: origin xyz=-0.386688019933338 0.197454290583016 1.93990580280716 rpy=0.780417755714486 0.206550528203247 1.54495729002601 -> xyz=-0.309528603559366 0.18089564105775 1.96606713304228 rpy=0.780417755714486 0.206550528203247 1.54495729002601
- joint pulley9: origin xyz=0.611640153384268 0.0201895234082593 1.06361661076598 rpy=1.3894765523934 0 0 -> xyz=0.598960734122778 0.0021129677620136 1.14249845306849 rpy=1.3894765523934 0 0
- joint tendon1: origin xyz=-0.0466759197978372 0.696113447385709 1.42131938536724 rpy=2.42029878837546 0.411085599759094 0.18803458251 -> xyz=-0.00737087429587602 0.627623395967135 1.47103362800014 rpy=0.724553090982325 -0.442232946231103 -2.97463015947492
- joint tendon2: origin xyz=-0.608609359052292 -0.0491036055084579 1.12579281338414 rpy=1.26117971092963 0.261335644435745 -0.0410112084771942 -> xyz=-0.555149044350002 -0.0669662547977792 1.21002859940116 rpy=1.25842678201526 0.282523150056682 -0.0447789619628604
- joint tendon3: origin xyz=-0.659713818386888 -0.128493991794642 1.09364244438357 rpy=2.31796632388059 0.687403267030743 0.278774820132193 -> xyz=-0.601682559529722 -0.146570547440898 1.17252428668608 rpy=2.31415645398289 0.701463240500334 0.283310410885007
- joint tendon4: origin xyz=0.0523061208957168 -0.0765710892010435 1.04170605862146 rpy=2.74376898576192 -1.46092772171524 -1.07377843875898 -> xyz=0.0622200803589977 -0.0954811833576393 1.12033347002897 rpy=2.73638977967294 -1.45380155814139 -1.06047574148992
- joint tendon5: axis 0 0 1 -> 0 -1 0; origin xyz=0.100914183112479 -0.409510270989431 1.76840273399034 rpy=2.03791065757841 0.0816434120527184 -0.340060952463484 -> xyz=0.104838833938817 -0.404324883250655 1.80075313592792 rpy=0.489632935594346 0.336016107582331 -0.202904079070031
- joint tendon6: origin xyz=0.410004431861938 -0.225457324111191 1.26383576024815 rpy=2.40337970476027 -0.626481292974809 -0.284482754458899 -> xyz=0.399200075389867 -0.241093665128849 1.32488833343546 rpy=2.4063038593005 -0.634839389370555 -0.289613435886281
- joint tendon7: axis 0 -1 0 -> 0 0 -1; origin xyz=0.286395054840697 0.089328919770948 2.01558559837794 rpy=2.49743103048459 1.49647330665931 0.868493247146079 -> xyz=-0.112898622615332 0.0957005775504391 2.00052094427155 rpy=-1.01637221920297 -1.45632726607529 -2.20607332712388
- joint tendon8: axis 0 -1 0 -> 0 0 -1; origin xyz=-0.101528663990072 0.629633422043848 1.48824784214199 rpy=2.27799917995113 -0.382849686510957 -0.142824130650291 -> xyz=-0.0724995267642046 0.564718142394954 1.53027492007169 rpy=-0.749025361344523 0.223845661453569 2.8362451546136
- joint tendon9: origin xyz=0.566770118853501 0.0612514071392795 1.08858398583577 rpy=0.391601755363025 -0.694514754049021 0.475091260901225 -> xyz=0.561786764721919 0.0442492543570693 1.16116779519199 rpy=0.397368609199379 -0.717419084371909 0.488556943438376
- joint tightener1: origin xyz=-0.0261159197978372 0.399512764329084 1.43386111414929 rpy=0.181319774401501 0 3.14159265358979 -> xyz=-0.00344000000000031 0.325880327868853 1.48698360655738 rpy=0.181319774401501 -7.82047468678116E-18 -3.14159265358979
- joint tightener2: origin xyz=-0.421921414642284 -0.075053824261462 1.26479790365546 rpy=-1.82448281699546 0.769136226420718 -0.178410499351035 -> xyz=-0.363890155785117 -0.0931303799077181 1.34367974595797 rpy=-1.82448281699546 0.769136226420718 -0.178410499351035
- joint tightener3: origin xyz=-0.0203759197978371 -0.338397727474194 1.56798570431322 rpy=1.57079632679489 1.3894765523934 -1.5707963267949 -> xyz=0.00229999999999975 -0.313669508196722 1.60307540983607 rpy=1.57079632679489 1.3894765523934 -1.5707963267949
- joint tightener4: origin xyz=-0.315855397464302 -0.0514025752621537 1.36829562546987 rpy=1.31710983659433 0.769136226420718 -0.178410499351035 -> xyz=-0.257824138607135 -0.0694791309084098 1.44717746777238 rpy=1.31710983659433 0.769136226420718 -0.178410499351035
- joint tightener5: origin xyz=0.107602569517075 0.0263707341619003 1.78619185869198 rpy=-0.785398163397445 0.181319774401482 1.5707963267949 -> xyz=0.0949231502555862 -0.00445692737460501 1.79552221432041 rpy=-0.785398163397445 0.181319774401482 1.5707963267949
- joint tightener6: origin xyz=-0.0249759197978372 -0.190856743867637 1.54093652398535 rpy=-1.5707963267949 1.3894765523934 -1.5707963267949 -> xyz=-0.00230000000000035 -0.166128524590164 1.5760262295082 rpy=-1.5707963267949 1.3894765523934 -1.5707963267949
- joint tightener7: origin xyz=-0.0476944936653156 0.124010188129215 1.65963797124096 rpy=-1.31710983659433 0.769136226420716 -2.96318215423875 -> xyz=0.0103367651918467 0.0931825265927212 1.66896832686939 rpy=-1.31710983659433 0.769136226420716 -2.96318215423875
- joint tightener8: origin xyz=-0.153760510843298 0.138612256800654 1.76479470944882 rpy=1.82448281699547 0.769136226420715 -2.96318215423875 -> xyz=-0.0957292519861357 0.10778459526416 1.77412506507724 rpy=1.82448281699547 0.769136226420716 -2.96318215423875
- joint tightener9: origin xyz=0.377375676777166 0.0487702268702811 1.24291636437404 rpy=0.785398163397445 0.181319774401485 1.5707963267949 -> xyz=0.364696257515673 0.0306936712240358 1.32179820667655 rpy=0.785398163397445 0.181319774401485 1.5707963267949
