Commit message: compact planning with w/wo Sting option

File: data/tensegrity/robots/tensegrity.URDF (robot description, URDF)
Before this commit: robot tensegrity, 46 links, 45 joints
Links:
- added link mid1, mass 0.00144131652160448; collision mesh filename=package://tensegrity/meshes/mid1.STL; visual mesh filename=package://tensegrity/meshes/mid1.STL
- added link mid2, mass 0.00144131652160447; collision mesh filename=package://tensegrity/meshes/mid2.STL; visual mesh filename=package://tensegrity/meshes/mid2.STL
- added link mid3, mass 0.00144131652160447; collision mesh filename=package://tensegrity/meshes/mid3.STL; visual mesh filename=package://tensegrity/meshes/mid3.STL
- added link mid4, mass 0.00144131652160447; collision mesh filename=package://tensegrity/meshes/mid4.STL; visual mesh filename=package://tensegrity/meshes/mid4.STL
- added link mid5, mass 0.00144131652160448; collision mesh filename=package://tensegrity/meshes/mid5.STL; visual mesh filename=package://tensegrity/meshes/mid5.STL
- added link mid6, mass 0.00144131652160448; collision mesh filename=package://tensegrity/meshes/mid6.STL; visual mesh filename=package://tensegrity/meshes/mid6.STL
- link attach1: mass 0.000125397117258045 -> 0.000125397117258048
- link attach2: mass 0.000125397117258046 -> 0.000125397117258051
- link attach3: mass 0.000125397117258043 -> 0.000125397117258047
- link attach4: mass 0.000125397117258046 -> 0.00012539711725805
- link attach5: mass 0.000125397117258043 -> 0.000125397117258046
- link attach7: mass 0.000125397117258042 -> 0.000125397117258045
- link attach8: mass 0.000125397117258044 -> 0.00012539711725805
- link attach9: mass 0.000125397117258043 -> 0.000125397117258047
- link detach1: mass 0.00144131652160448 -> 0.00144131652160447
- link detach2: mass 0.00144131652160447 -> 0.00144131652160448
- link detach5: mass 0.00144131652160446 -> 0.00144131652160448
- link detach8: mass 0.00144131652160447 -> 0.00144131652160448
- link detach9: mass 0.00144131652160446 -> 0.00144131652160448
- link pulley3: mass 0.00115149136839394 -> 0.00115149136839398
- link pulley4: mass 0.00115149136839396 -> 0.00115149136839393
- link pulley6: mass 0.00115149136839394 -> 0.00115149136839398
- link pulley7: mass 0.00115149136839396 -> 0.00115149136839393
- link pulley8: mass 0.00115149136839396 -> 0.00115149136839392
- link tendon1: mass 0.0103991743382068 -> 0.0123205724051423
- link tendon2: mass 0.0111099282601549 -> 0.0106761371465473
- link tendon3: mass 0.0109723265019277 -> 0.0118735866023895
- link tendon4: mass 0.0142485049847973 -> 0.0112680132024836
- link tendon5: mass 0.00943206645572571 -> 0.00968829475255249
- link tendon6: mass 0.0117808467872556 -> 0.0108793353593815
- link tendon7: mass 0.0071673551436059 -> 0.00905708595659323
- link tendon8: mass 0.00906487710637413 -> 0.0073184029183905
- link tendon9: mass 0.0109763477405243 -> 0.0109928096860291
- link tensegrity: mass 2.981 -> 3.00545265429648
- link tightener1: mass 0.00856462996419102 -> 0.0085646299641912
- link tightener2: mass 0.00856464520084429 -> 0.00856464520084457
- link tightener3: mass 0.00856463183459565 -> 0.00856463183459577
- link tightener4: mass 0.00856463280589177 -> 0.0085646328058922
- link tightener5: mass 0.00856464027785648 -> 0.00856464027785653
- link tightener6: mass 0.00856463401560627 -> 0.00856463401560592
- link tightener7: mass 0.00856463670998778 -> 0.00856463670998783
- link tightener9: mass 0.00856463882730577 -> 0.00856463882730581
Joints:
- removed joint detach
- added joint detach1: type fixed, parent tensegrity, child detach1, origin xyz=0.0210000000000689 0.380483606557384 1.49506967213115 rpy=0 -0.181319774401501 -1.5707963267949, axis 0 0 0
- added joint mid1: type fixed, parent tensegrity, child mid1, origin xyz=0 -0.0407921561087422 1.288 rpy=3.14159265358979 1.5707963267949 0, axis 0 0 0
- added joint mid2: type fixed, parent tensegrity, child mid2, origin xyz=0.0353270434653114 -0.020396078054371 1.288 rpy=2.09439510239319 1.5707963267949 0, axis 0 0 0
- added joint mid3: type fixed, parent tensegrity, child mid3, origin xyz=-0.0353270434653113 0.0203960780543712 1.288 rpy=1.0471975511966 1.5707963267949 0, axis 0 0 0
- added joint mid4: type fixed, parent tensegrity, child mid4, origin xyz=0 0.0407921561087424 1.288 rpy=0 1.5707963267949 0, axis 0 0 0
- added joint mid5: type fixed, parent tensegrity, child mid5, origin xyz=0.0353270434653114 0.0203960780543712 1.288 rpy=1.0471975511966 1.5707963267949 0, axis 0 0 0
- added joint mid6: type fixed, parent tensegrity, child mid6, origin xyz=-0.0353270434653115 -0.0203960780543711 1.288 rpy=2.0943951023932 1.5707963267949 0, axis 0 0 0
- joint attach1: origin xyz=0.318156761076164 0.0650930969857314 1.97852563931339 rpy=-0.531711673196898 0.769136226420716 -2.96318215423882 -> xyz=0.596432559529796 -0.0939848544548516 1.15754607630531 rpy=-2.10250799999178 -0.769136226420718 2.96318215423875
- joint attach2: origin xyz=-0.328656761076175 0.166626629046522 1.94923615843558 rpy=0.531711673196865 0.769136226420715 -0.178410499351044 -> xyz=-0.0304246212023898 0.621142144807008 1.46713897167455 rpy=-2.35619449019234 -0.181319774401499 -1.5707963267949
- joint attach3: origin xyz=-0.601682559529722 -0.146570547440898 1.17252428668608 rpy=-2.6098809803929 -0.769136226420708 0.178410499351032 -> xyz=-0.596432559529653 -0.0374265613533095 1.14911892837741 rpy=-2.6098809803929 -0.769136226420706 0.178410499351035
- joint attach4: origin xyz=0.546741434032771 -0.0384451766288569 1.09684449111531 rpy=1.03908465359801 -0.769136226420713 2.96318215423876 -> xyz=-0.323406761076112 0.0558598630161561 1.97488089887448 rpy=0.531711673196865 0.769136226420715 -0.178410499351044
- joint attach5: origin xyz=0.0239999999999999 -0.59522390710731 1.69768777941467 rpy=-2.35619449019234 0.181319774401499 1.5707963267949 -> xyz=0.0324246212025278 0.621142144807008 1.46713897167455 rpy=2.35619449019234 -0.181319774401488 -1.57079632679491
- joint attach6: origin xyz=0.591182559529726 -0.0450370153801445 1.14323480580828 rpy=2.60988098039293 -0.769136226420713 2.96318215423875 -> xyz=0.596432559529791 -0.15580378141051 1.16887954624718 rpy=2.60988098039293 -0.769136226420717 2.96318215423874
- joint attach7: origin xyz=0.273715635579209 0.0585012582344451 2.02491595400636 rpy=-2.10250799999181 0.769136226420727 -2.96318215423883 -> xyz=-0.0304246212023898 -0.596562773225779 1.69038487331389 rpy=2.35619449019234 0.181319774401488 1.57079632679491
- joint attach8: origin xyz=-0.0240000000000005 0.622481010925478 1.47444187777533 rpy=-2.35619449019234 -0.181319774401499 -1.5707963267949 -> xyz=0.278965635579294 0.120432129567981 2.0101663334026 rpy=2.6098809803929 0.769136226420707 -2.96318215423875
- joint attach9: origin xyz=0.0239999999999996 0.608469808746655 1.39801713861811 rpy=0.785398163397449 -0.181319774401489 -1.57079632679489 -> xyz=0.323406761076249 0.112418156117712 1.96645375094658 rpy=1.039084653598 0.76913622642071 -2.96318215423875
- joint detach2: origin xyz=-0.421300155349653 -0.0844233171255465 1.31741827022436 rpy=1.31710983659433 -0.769136226420714 0.178410499351039 -> xyz=-0.412814873975346 0.0389266585893259 1.30537268321449 rpy=1.31710983659433 -0.769136226420713 0.178410499351047
- joint detach3: origin xyz=-0.0110000000000003 -0.366245901639344 1.63654508196721 rpy=1.5707963267949 0.181319774401488 1.5707963267949 -> xyz=-0.0144999999999317 -0.354442622950813 1.63438114754098 rpy=1.5707963267949 0.181319774401488 1.5707963267949
- joint detach4: origin xyz=-0.32831561362362 -0.09814741615855 1.41446863913521 rpy=1.31710983659433 -0.769136226420712 0.178410499351048 -> xyz=-0.319830332249315 0.0252025595563105 1.40242305212534 rpy=1.31710983659434 -0.769136226420714 0.178410499351044
- joint detach5: origin xyz=0.124586279726341 -0.0164765829315123 1.85994591128273 rpy=0.253686490200554 0.769136226420711 -2.96318215423876 -> xyz=0.11928297886751 0.098813098096445 1.82888962598058 rpy=0.253686490200554 0.769136226420711 -2.96318215423876
- joint detach6: origin xyz=0.0199999999999994 -0.236901639344262 1.61283196721312 rpy=1.5707963267949 0.181319774401488 1.5707963267949 -> xyz=0.0165000000000686 -0.225098360655731 1.61066803278689 rpy=1.5707963267949 0.181319774401488 1.5707963267949
- joint detach7: origin xyz=-0.0270055439226141 0.0839596778251951 1.74232551541019 rpy=1.31710983659433 0.769136226420715 -0.178410499351034 -> xyz=-0.136488248106043 -0.010887703387596 1.87102161788576 rpy=1.31710983659432 0.769136226420714 -0.178410499351051
- joint detach8: origin xyz=-0.119990085648646 0.131219185349568 1.82819555645219 rpy=1.31710983659433 0.769136226420715 -0.178410499351032 -> xyz=-0.111504804274339 0.0150988887083267 1.84085757477261 rpy=1.31710983659432 0.769136226420715 -0.178410499351043
- joint detach9: origin xyz=0.425896349427369 0.00228884459815839 1.29684824326267 rpy=0.253686490200553 -0.769136226420708 2.96318215423877 -> xyz=0.414229087537839 -0.115771215902692 1.32388427689438 rpy=0.253686490200553 -0.769136226420708 2.96318215423877
- joint pulley1: axis 0 0 1 -> 0 0 0; origin xyz=0 0.621786885245901 1.47065573770492 rpy=1.5707963267949 -1.35303842246507 -1.5707963267949 -> xyz=0.000750000000068907 0.621786885245909 1.47065573770492 rpy=1.5707963267949 -1.35303842246507 -1.5707963267949; type continuous -> fixed
- joint pulley2: axis 0 0 1 -> 0 0 0; origin xyz=-0.573455270689443 -0.0936279273956821 1.13412039602351 rpy=0.631420863095884 0.532284485238217 -2.35588130681373 -> xyz=-0.574388773476476 0.0239340226723326 1.11545830548531 rpy=0.631420863095884 0.532284485238218 -2.35588130681373; type continuous -> fixed
- joint pulley3: axis 0 0 1 -> 0 0 0; origin xyz=-0.0350000000000004 -0.60298527630066 1.65535303836004 rpy=2.98449472353879 -0.0909133937987541 -0.520440071048006 -> xyz=-0.0339999999999311 -0.602184426229502 1.65972131147541 rpy=2.98449472353879 -0.0909133937987541 -0.520440071048006; type continuous -> fixed
- joint pulley4: axis 0 0 1 -> 0 0 0; origin xyz=-0.572811013144504 -0.162596564002146 1.14610965089734 rpy=0.745639043009377 0.327890658213947 -2.08475010947139 -> xyz=-0.574035220085884 -0.0449821918735116 1.12773349887161 rpy=0.745639043009377 0.327890658213947 -2.08475010947139; type continuous -> fixed
- joint pulley5: axis 0 0 -1 -> 0 0 0; origin xyz=0.276437460986168 0.0428433090569649 2.02501938885851 rpy=1.36772787967172 0.464271853741143 -0.0919392370595983 -> xyz=0.276437460986239 0.152043395021608 2.00694124557237 rpy=1.36772787967172 0.464271853741143 -0.0919392370595982; type continuous -> fixed
- joint pulley6: axis 0 0 1 -> 0 0 0; origin xyz=0.0349999999999996 -0.603075440235086 1.65486123508135 rpy=3.12170686669581 0.180237919378081 1.4603031742211 -> xyz=0.0360000000000689 -0.602274590163928 1.65922950819672 rpy=3.12170686669581 0.180237919378081 1.4603031742211; type continuous -> fixed
- joint pulley7: axis 0 0 1 -> 0 0 0; origin xyz=-0.310210537417404 0.111920210362038 1.97801932924749 rpy=2.37738677488523 -0.271358663823417 -1.66506917334562 -> xyz=-0.301362975022931 -0.00550072100945849 2.00854152176658 rpy=2.37738677488523 -0.271358663823428 -1.66506917334561; type continuous -> fixed
- joint pulley8: axis 0 0 -1 -> 0 0 0; origin xyz=-0.309528603559366 0.18089564105775 1.96606713304228 rpy=0.780417755714486 0.206550528203247 1.54495729002601 -> xyz=-0.301009421632338 0.0634154935363862 1.99626632838028 rpy=0.780417755714485 0.206550528203247 1.54495729002601; type continuous -> fixed
- joint pulley9: axis 0 0 -1 -> 0 0 0; origin xyz=0.598960734122778 0.0021129677620136 1.14249845306849 rpy=1.3894765523934 0 0 -> xyz=0.598960734122845 -0.124192515956886 1.16565445841695 rpy=1.3894765523934 0 0; type continuous -> fixed
- joint tendon1: origin xyz=-0.00737087429587602 0.627623395967135 1.47103362800014 rpy=0.724553090982325 -0.442232946231103 -2.97463015947492 -> xyz=0.0070000000000689 0.619377049180335 1.4741475409836 rpy=-2.05407776195157 1.2043856781213 1.75162768833035
- joint tendon2: origin xyz=-0.555149044350002 -0.0669662547977792 1.21002859940116 rpy=1.25842678201526 0.282523150056682 -0.0447789619628604 -> xyz=-0.580575957811856 0.0272354977564193 1.11682998776229 rpy=0.542760383124674 0.679222116277311 -0.385370645633379
- joint tendon3: axis 0 -1 0 -> 0 1 0; origin xyz=-0.601682559529722 -0.146570547440898 1.17252428668608 rpy=2.31415645398289 0.701463240500334 0.283310410885007 -> xyz=-0.0369999999999311 -0.604098360655731 1.66591803278689 rpy=-1.97723117907901 -0.944746282793038 2.83859847552446
- joint tendon4: axis 0 1 0 -> 0 -1 0; origin xyz=0.0622200803589977 -0.0954811833576393 1.12033347002897 rpy=2.73638977967294 -1.45380155814139 -1.06047574148992 -> xyz=-0.572090676437616 -0.0490487333110664 1.12218872739419 rpy=1.440424684019 0.282232816368081 -0.0185464264423147
- joint tendon5: axis 0 -1 0 -> 0 1 0; origin xyz=0.104838833938817 -0.404324883250655 1.80075313592792 rpy=0.489632935594346 0.336016107582331 -0.202904079070031 -> xyz=0.276437460986242 0.158464199079938 2.01007744952691 rpy=-0.904840677620968 -0.402289800523352 0.935725152760631
- joint tendon6: axis 0 -1 0 -> 0 1 0; origin xyz=0.399200075389867 -0.241093665128849 1.32488833343546 rpy=2.4063038593005 -0.634839389370555 -0.289613435886281 -> xyz=0.0387071067812556 -0.604225871714633 1.66522251792014 rpy=-0.843481301503022 0.696282568469085 -1.5232985820643
- joint tendon7: axis 0 0 -1 -> 0 -1 0; origin xyz=-0.112898622615332 0.0957005775504391 2.00052094427155 rpy=-1.01637221920297 -1.45632726607529 -2.20607332712388 -> xyz=-0.307550159358307 -0.0088021960935663 2.0071698394896 rpy=-2.65608974352876 0.398388925164006 0.646068565378626
- joint tendon8: axis 0 0 -1 -> 0 -1 0; origin xyz=-0.0724995267642046 0.564718142394954 1.53027492007169 rpy=-0.749025361344523 0.223845661453569 2.8362451546136 -> xyz=-0.299064877984069 0.0674820349739192 2.0018110998577 rpy=0.182977508146443 1.49011189347165 -1.30905774743622
- joint tendon9: axis 0 1 0 -> 0 0 -1; origin xyz=0.561786764721919 0.0442492543570693 1.16116779519199 rpy=0.397368609199379 -0.717419084371909 0.488556943438376 -> xyz=0.603203374809965 -0.130340056940491 1.16678150759728 rpy=-0.157059449593044 -0.40457084948561 -0.346816167000894
- joint tightener1: origin xyz=-0.00344000000000031 0.325880327868853 1.48698360655738 rpy=0.181319774401501 -7.82047468678116E-18 -3.14159265358979 -> xyz=0.0440793418117183 0.335790163934433 1.48974180327869 rpy=0.181319774401501 0 3.14159265358979
- joint tightener2: origin xyz=-0.363890155785117 -0.0931303799077181 1.34367974595797 rpy=-1.82448281699546 0.769136226420718 -0.178410499351035 -> xyz=-0.390243560110425 0.035800670929021 1.36207638688557 rpy=-1.82448281699546 0.769136226420719 -0.178410499351027
- joint tightener3: origin xyz=0.00229999999999975 -0.313669508196722 1.60307540983607 rpy=1.57079632679489 1.3894765523934 -1.5707963267949 -> xyz=-0.0011999999999311 -0.296182413771663 1.64716410669998 rpy=1.57079632679489 1.3894765523934 -1.5707963267949
- joint tightener4: origin xyz=-0.257824138607135 -0.0694791309084098 1.44717746777238 rpy=1.31710983659433 0.769136226420718 -0.178410499351035 -> xyz=-0.297259018384395 0.0482405063222401 1.45433003448494 rpy=1.31710983659433 0.769136226420719 -0.178410499351027
- joint tightener5: origin xyz=0.0949231502555862 -0.00445692737460501 1.79552221432041 rpy=-0.785398163397445 0.181319774401482 1.5707963267949 -> xyz=0.0982819074662917 0.0689332335343484 1.79389398750648 rpy=-0.785398163397444 0.181319774401482 1.57079632679491
- joint tightener6: origin xyz=-0.00230000000000035 -0.166128524590164 1.5760262295082 rpy=-1.5707963267949 1.3894765523934 -1.5707963267949 -> xyz=0.00320000000006892 -0.166838151476581 1.62345099194588 rpy=-1.5707963267949 1.3894765523934 -1.5707963267949
- joint tightener7: origin xyz=0.0103367651918467 0.0931825265927212 1.66896832686939 rpy=-1.31710983659433 0.769136226420716 -2.96318215423875 -> xyz=0.0366901695172931 -0.0231488885293931 1.73038788074873 rpy=-1.31710983659433 0.769136226420714 -2.96318215423875
- joint tightener8: origin xyz=-0.0957292519861357 0.10778459526416 1.77412506507724 rpy=1.82448281699547 0.769136226420716 -2.96318215423875 -> xyz=-0.0562943722087432 -0.00205331543125625 1.8210546431022 rpy=1.82448281699547 0.769136226420716 -2.96318215423875
- joint tightener9: origin xyz=0.364696257515673 0.0306936712240358 1.32179820667655 rpy=0.785398163397445 0.181319774401485 1.5707963267949 -> xyz=0.374418975757055 -0.134685129399173 1.34870291695999 rpy=0.785398163397445 0.181319774401485 1.5707963267949

Commit message: multi plan

File: data/tensegrity/robots/tensegrity.URDF (robot description, URDF)
Before this commit: robot tensegrity, 52 links, 51 joints
Links:
- removed link mid1
- removed link mid2
- removed link mid3
- removed link mid4
- removed link mid5
- removed link mid6
- link tensegrity: geometry collision mesh filename=package://tensegrity/meshes/tensegrity.STL scale=1 1 1; visual mesh filename=package://tensegrity/meshes/tensegrity.STL scale=1 1 1
Joints:
- removed joint mid1
- removed joint mid2
- removed joint mid3
- removed joint mid4
- removed joint mid5
- removed joint mid6

Commit message: fixed cleaned planning

File: data/tensegrity/robots/tensegrity.URDF (robot description, URDF)
Before this commit: robot tensegrity, 46 links, 45 joints
Links:
- link tensegrity: geometry collision mesh filename=package://tensegrity/meshes/tensegrityNoPole.stl scale=0.001 0.001 0.001; visual mesh filename=package://tensegrity/meshes/tensegrityNoPole.stl scale=0.001 0.001 0.001
