Commit message: Almost DONE!

File: data/tensegrity/robots/tensegrity.URDF (robot description, URDF)
Before this commit: robot tensegrity, 46 links, 45 joints
Links:
- link attach1: mass 0.000125397117258048 -> 0.000125397117258047
- link attach2: mass 0.000125397117258051 -> 0.000125397117258047
- link attach3: mass 0.000125397117258047 -> 0.000125397117258045
- link attach4: mass 0.00012539711725805 -> 0.000125397117258047
- link attach5: mass 0.000125397117258046 -> 0.00012539711725805
- link attach6: mass 0.000125397117258046 -> 0.000125397117258042
- link attach7: mass 0.000125397117258045 -> 0.000125397117258043
- link attach8: mass 0.00012539711725805 -> 0.000125397117258044
- link attach9: mass 0.000125397117258047 -> 0.000125397117258046
- link detach1: mass 0.00144131652160447 -> 0.00144131652160448
- link detach2: mass 0.00144131652160448 -> 0.00144131652160445
- link detach3: mass 0.00144131652160448 -> 0.00144131652160447
- link detach6: mass 0.00144131652160448 -> 0.00144131652160446
- link pulley2: mass 0.00115149136839393 -> 0.00115149136839394
- link pulley3: mass 0.00115149136839398 -> 0.00115149136839397
- link pulley4: mass 0.00115149136839393 -> 0.00115149136839394
- link pulley5: mass 0.00115149136839394 -> 0.00115149136839393
- link pulley6: mass 0.00115149136839398 -> 0.00115149136839395
- link pulley7: mass 0.00115149136839392 -> 0.00115149136839397
- link pulley8: mass 0.00115149136839392 -> 0.00115149136839394
- link pulley9: mass 0.00115149136839395 -> 0.00115149136839394
- link tendon1: mass 0.0123205724051423 -> 0.0110584061406361
- link tendon2: mass 0.0111536592298929 -> 0.0124281405376012
- link tendon3: mass 0.0118735866023895 -> 0.0112594680704658
- link tendon4: mass 0.0112680132024836 -> 0.0109830079169499
- link tendon5: mass 0.00968829475255249 -> 0.00907291958356732
- link tendon6: mass 0.0108793353593815 -> 0.00755238873922986
- link tendon7: mass 0.00905708595659323 -> 0.0111589371055509
- link tendon8: mass 0.0073184029183905 -> 0.00952530892568425
- link tendon9: mass 0.0109928096860291 -> 0.0118877866011838
- link tensegrity: mass 3.00545265429648 -> 3.25616160799484; geometry collision mesh filename=package://tensegrity/meshes/tensegrity.STL; visual mesh filename=package://tensegrity/meshes/tensegrity.STL
- link tightener1: mass 0.0085646299641912 -> 0.00856463562467956
- link tightener2: mass 0.00856464520084458 -> 0.00856462494552237
- link tightener3: mass 0.00856463183459577 -> 0.0085646455096891
- link tightener4: mass 0.0085646328058922 -> 0.00856462494552187
- link tightener5: mass 0.00856464027785653 -> 0.00856464550968897
- link tightener6: mass 0.00856463401560592 -> 0.00856464550968905
- link tightener7: mass 0.00856463670998783 -> 0.00856464550968895
- link tightener8: mass 0.00856465792468904 -> 0.00856463562467937
- link tightener9: mass 0.00856463882730581 -> 0.0085646249455224
Joints:
- joint attach1: origin xyz=0.596432559529796 -0.0939848544548516 1.15754607630531 rpy=-2.10250799999178 -0.769136226420718 2.96318215423875 -> xyz=-0.423575378797548 0.323406761076181 1.97890676107617 rpy=0.785398163397434 0.785398163397451 -1.57079632679489
- joint attach2: origin xyz=-0.0304246212023898 0.621142144807008 1.46713897167455 rpy=-2.35619449019234 -0.181319774401499 -1.5707963267949 -> xyz=-0.366424621202465 0.596432559529732 1.14794969146418 rpy=-2.35619449019236 -0.785398163397448 -1.57079632679488
- joint attach3: origin xyz=-0.596432559529653 -0.0374265613533095 1.14911892837741 rpy=-2.6098809803929 -0.769136226420706 0.178410499351035 -> xyz=-0.366424621202454 -0.323406761076168 1.97890676107618 rpy=0.785398163397439 0.785398163397456 1.57079632679489
- joint attach4: origin xyz=-0.323406761076112 0.0558598630161561 1.97488089887448 rpy=0.531711673196865 0.769136226420715 -0.178410499351044 -> xyz=-0.303575378797548 0.596432559529733 1.14794969146418 rpy=2.35619449019236 -0.785398163397454 -1.57079632679489
- joint attach5: origin xyz=0.0324246212025278 0.621142144807008 1.46713897167455 rpy=2.35619449019234 -0.181319774401488 -1.57079632679491 -> xyz=0.224 -0.0304246212024516 1.58142462120246 rpy=2.35619449019234 0 3.14159265358979
- joint attach6: origin xyz=0.596432559529791 -0.15580378141051 1.16887954624718 rpy=2.60988098039293 -0.769136226420717 2.96318215423874 -> xyz=-0.486424621202465 0.278965635579226 2.02334788657313 rpy=-2.35619449019237 0.785398163397443 -1.5707963267949
- joint attach7: origin xyz=-0.0304246212023898 -0.596562773225779 1.69038487331389 rpy=2.35619449019234 0.181319774401488 1.57079632679491 -> xyz=-1.014 -0.0304246212024514 1.58142462120246 rpy=-2.35619449019234 0 0
- joint attach8: origin xyz=0.278965635579294 0.120432129567981 2.0101663334026 rpy=2.6098809803929 0.769136226420707 -2.96318215423875 -> xyz=-1.014 0.032424621202466 1.58142462120246 rpy=2.35619449019234 0 0
- joint attach9: origin xyz=0.323406761076249 0.112418156117712 1.96645375094658 rpy=1.039084653598 0.76913622642071 -2.96318215423875 -> xyz=-0.423575378797541 -0.596432559529721 1.14794969146418 rpy=-2.35619449019236 -0.785398163397451 1.57079632679491
- joint detach1: origin xyz=0.0210000000000689 0.380483606557384 1.49506967213115 rpy=0 -0.181319774401501 -1.5707963267949 -> xyz=-0.315000000000004 0.414229087537811 1.30763234817594 rpy=-9.61372600496381E-31 -0.785398163397456 -1.57079632679489
- joint detach2: origin xyz=-0.412814873975346 0.0389266585893259 1.30537268321449 rpy=1.31710983659433 -0.769136226420713 0.178410499351047 -> xyz=-0.77225 0.0210000000000074 1.5655 rpy=-6.12303176911189E-17 0 0
- joint detach3: origin xyz=-0.0144999999999317 -0.354442622950813 1.63438114754098 rpy=1.5707963267949 0.181319774401488 1.5707963267949 -> xyz=-0.439499999999991 -0.319830332249379 1.40839506449503 rpy=1.57079632679491 -0.785398163397444 1.57079632679489
- joint detach4: origin xyz=-0.319830332249315 0.0252025595563105 1.40242305212534 rpy=1.31710983659434 -0.769136226420714 0.178410499351044 -> xyz=-0.15575 0.0165000000000074 1.57 rpy=1.5707963267949 0 3.14159265358979
- joint detach5: origin xyz=0.11928297886751 0.098813098096445 1.82888962598058 rpy=0.253686490200554 0.769136226420711 -2.96318215423876 -> xyz=-0.314999999999997 -0.148097580200831 1.86995901591455 rpy=-3.14159265358976 0.785398163397454 1.57079632679492
- joint detach6: origin xyz=0.0165000000000686 -0.225098360655731 1.61066803278689 rpy=1.5707963267949 0.181319774401488 1.5707963267949 -> xyz=-0.350499999999991 -0.111504804274401 1.83973020101882 rpy=1.5707963267949 0.785398163397447 1.57079632679491
- joint detach7: origin xyz=-0.136488248106043 -0.010887703387596 1.87102161788576 rpy=1.31710983659432 0.769136226420714 -0.178410499351051 -> xyz=-0.470500000000004 -0.412814873975416 1.315410522769 rpy=1.57079632679489 -0.785398163397444 1.57079632679492
- joint detach8: origin xyz=-0.111504804274339 0.0150988887083267 1.84085757477261 rpy=1.31710983659432 0.769136226420715 -0.178410499351043 -> xyz=-0.435000000000005 0.119282978867482 1.84114441458119 rpy=0 0.785398163397453 -1.5707963267949
- joint detach9: origin xyz=0.414229087537839 -0.115771215902692 1.32388427689438 rpy=0.253686490200553 -0.769136226420708 2.96318215423877 -> xyz=-0.0242500000000002 -0.0144999999999926 1.57 rpy=1.5707963267949 0 3.14159265358979
- joint pulley1: axis 0 0 -1 -> 0 0 0; origin xyz=0.000750000000068907 0.621786885245909 1.47065573770492 rpy=1.5707963267949 -1.35303842246507 -1.5707963267949 -> xyz=-0.335249999999995 0.59896073412282 1.15047786605722 rpy=1.5707963267949 -1.35303842246507 -1.5707963267949
- joint pulley2: axis 0 0 -1 -> 0 0 0; origin xyz=-0.574388773476476 0.0239340226723326 1.11545830548531 rpy=0.631420863095884 0.532284485238218 -2.35588130681373 -> xyz=-1.014 0.000750000000007453 1.585 rpy=1.5707963267949 -0.187598613267775 3.14159265358979
- joint pulley3: axis 0 0 -1 -> 0 0 0; origin xyz=-0.0339999999999311 -0.602184426229502 1.65972131147541 rpy=2.98449472353879 -0.0909133937987541 -0.520440071048006 -> xyz=-0.419999999999997 -0.574035220085944 1.12555235202041 rpy=-0.520114409814359 0.618304773840794 -2.35017143556008
- joint pulley4: axis 0 0 -1 -> 0 0 0; origin xyz=-0.574035220085884 -0.0449821918735116 1.12773349887161 rpy=0.745639043009377 0.327890658213947 -2.08475010947139 -> xyz=0.224 0.0360000000000074 1.54975 rpy=3.14159265358979 -3.08271311160171E-17 -0.527600849438056
- joint pulley5: axis 0 0 1 -> 0 0 0; origin xyz=0.276437460986239 0.152043395021608 2.00694124557237 rpy=1.36772787967172 0.464271853741143 -0.0919392370595982 -> xyz=-0.30000000000001 -0.301362975022985 2.00095054712935 rpy=3.01454229621802 -0.777239250993921 -1.39062986286711
- joint pulley6: axis 0 0 -1 -> 0 0 0; origin xyz=0.0360000000000689 -0.602274590163928 1.65922950819672 rpy=3.12170686669581 0.180237919378081 1.4603031742211 -> xyz=-0.37000000000001 -0.301009421632392 2.00130410051995 rpy=0.215724281605467 0.761379037634035 1.87834102549842
- joint pulley7: axis 0 0 -1 -> 0 0 0; origin xyz=-0.301362975022931 -0.00550072100945849 2.00854152176658 rpy=2.37738677488523 -0.271358663823428 -1.66506917334561 -> xyz=-0.489999999999997 -0.574388773476538 1.12590590541101 rpy=0.785398163397448 0 0
- joint pulley8: axis 0 0 1 -> 0 0 0; origin xyz=-0.301009421632338 0.0634154935363862 1.99626632838028 rpy=0.780417755714485 0.206550528203247 1.54495729002601 -> xyz=-0.455250000000007 0.276437460986177 2.02587606116618 rpy=1.5707963267949 0.653955584294836 1.5707963267949
- joint pulley9: axis 0 0 1 -> 0 0 0; origin xyz=0.598960734122845 -0.124192515956886 1.16565445841695 rpy=1.3894765523934 0 0 -> xyz=0.224 -0.0340000000000102 1.55025 rpy=3.14159265358979 6.08689601468759E-17 1.4621001866288
- joint tendon1: origin xyz=0.0070000000000689 0.619377049180335 1.4741475409836 rpy=-2.05407776195157 1.2043856781213 1.75162768833035 -> xyz=-0.303575378797548 0.596432559529733 1.14794969146418 rpy=1.89878694392289 -0.0999397467306176 -0.0165515790073519
- joint tendon2: axis 0 -1 0 -> 0 1 0; origin xyz=-0.580575957811856 0.0272354977564193 1.11682998776229 rpy=0.542760383124674 0.679222116277311 -0.385370645633379 -> xyz=-0.645783745357682 0.338571529284564 1.34139404716458 rpy=-0.622554031987558 0.718383702173134 -1.26337260624258
- joint tendon3: axis 0 1 0 -> 0 -1 0; origin xyz=-0.0369999999999311 -0.604098360655731 1.66591803278689 rpy=-1.97723117907901 -0.944746282793038 2.83859847552446 -> xyz=-0.413581774467045 -0.552517068226954 1.18643801555917 rpy=1.28738486601303 0.0519432689767225 0.00352083993720131
- joint tendon4: axis 0 -1 0 -> 0 1 0; origin xyz=-0.572090676437616 -0.0490487333110664 1.12218872739419 rpy=1.440424684019 0.282232816368081 -0.0185464264423147 -> xyz=-0.334742206728285 0.584755860469229 1.20469041170867 rpy=-0.620518440095981 -0.655602260092983 1.16819224375592
- joint tendon5: origin xyz=0.276437460986242 0.158464199079938 2.01007744952691 rpy=-0.904840677620968 -0.402289800523352 0.935725152760631 -> xyz=-0.0252798809574738 -0.157939522547366 1.78920469338102 rpy=-0.996875567930223 0.807564348851391 -1.93268509594004
- joint tendon6: origin xyz=0.0387071067812556 -0.604225871714633 1.66522251792014 rpy=-0.843481301503022 0.696282568469085 -1.5232985820643 -> xyz=-0.402797935908687 -0.161471710808598 2.00478467391487 rpy=0.0395380632265221 -0.201072093145439 0.193324657373221
- joint tendon7: axis 0 -1 0 -> 0 1 0; origin xyz=-0.307550159358307 -0.0088021960935663 2.0071698394896 rpy=-2.65608974352876 0.398388925164006 0.646068565378626 -> xyz=-0.632248236732676 -0.433157901561712 1.2506374332294 rpy=0.694492436909307 -0.62782945974723 0.301898503624934
- joint tendon8: axis 0 -1 0 -> 0 1 0; origin xyz=-0.299064877984069 0.0674820349739192 2.0018110998577 rpy=0.182977508146443 1.49011189347165 -1.30905774743622 -> xyz=-0.956042633236307 0.0557443592956697 1.63418830440659 rpy=-2.08142941879277 -0.840637055189645 -2.08447812649533
- joint tendon9: axis 0 0 -1 -> 0 1 0; origin xyz=0.603203374809965 -0.130340056940491 1.16678150759728 rpy=-0.157059449593044 -0.40457084948561 -0.346816167000894 -> xyz=-0.321653388057719 -0.51267513693146 1.20604467417496 rpy=-2.50967163899156 -0.748466312512797 -1.31767322172929
- joint tightener1: origin xyz=0.0440793418117183 0.335790163934433 1.48974180327869 rpy=0.181319774401501 0 3.14159265358979 -> xyz=-0.291920658188362 0.374418975756998 1.32863341957718 rpy=0.785398163397452 3.92523114670945E-15 3.14159265358979
- joint tightener2: origin xyz=-0.390243560110425 0.035800670929021 1.36207638688557 rpy=-1.82448281699546 0.769136226420719 -0.178410499351027 -> xyz=-0.72925 0.0440793418116571 1.5522 rpy=3.14159265358979 -6.12303176911189E-17 -1.5707963267949
- joint tightener3: origin xyz=-0.0011999999999311 -0.296182413771663 1.64716410669998 rpy=1.57079632679489 1.3894765523934 -1.5707963267949 -> xyz=-0.452800000000002 -0.297259018384463 1.46360549656063 rpy=1.5707963267949 0.785398163397448 1.57079632679491
- joint tightener4: origin xyz=-0.297259018384395 0.0482405063222401 1.45433003448494 rpy=1.31710983659433 0.769136226420719 -0.178410499351027 -> xyz=-0.21075 0.00320000000000739 1.59307934181165 rpy=1.5707963267949 1.5707963267949 0
- joint tightener5: origin xyz=0.0982819074662917 0.0689332335343484 1.79389398750648 rpy=-0.785398163397444 0.181319774401482 1.57079632679491 -> xyz=-0.332799999999999 0.0366901695172307 1.72417434542787 rpy=-1.5707963267949 0.785398163397446 -1.57079632679489
- joint tightener6: origin xyz=0.00320000000006892 -0.166838151476581 1.62345099194588 rpy=-1.5707963267949 1.3894765523934 -1.5707963267949 -> xyz=-0.337199999999998 -0.0562943722088002 1.8171588871539 rpy=1.57079632679489 0.785398163397447 -1.57079632679489
- joint tightener7: origin xyz=0.0366901695172931 -0.0231488885293931 1.73038788074873 rpy=-1.31710983659433 0.769136226420714 -2.96318215423875 -> xyz=-0.457200000000001 -0.390243560110494 1.3706209548346 rpy=-1.57079632679489 0.785398163397448 1.57079632679491
- joint tightener8: origin xyz=-0.0562943722087432 -0.00205331543125625 1.8210546431022 rpy=1.82448281699547 0.769136226420716 -2.96318215423875 -> xyz=-0.411920658188356 0.0982819074662237 1.80133430280039 rpy=-0.78539816339745 0 3.14159265358979
- joint tightener9: origin xyz=0.374418975757055 -0.134685129399173 1.34870291695999 rpy=0.785398163397445 0.181319774401485 1.5707963267949 -> xyz=-0.0792500000000005 -0.00119999999999264 1.59307934181165 rpy=1.5707963267949 1.5707963267949 0

Commit message: added sphere cushion

File: data/tensegrity/robots/tensegrity.URDF (robot description, URDF)
Before this commit: robot tensegrity, 46 links, 45 joints
Links:
- added link ball1, mass 0.000125397117258046; collision sphere radius=0.15; visual sphere radius=0.15
Joints:
- added joint ball1: type fixed, parent tensegrity, child ball1, origin xyz=-0.453575378797541 -0.586432559529721 1.13794969146418 rpy=0 0 0, axis 0 0 0

Commit message: clean up

File: data/tensegrity/robots/tensegrity.URDF (robot description, URDF)
Before this commit: robot tensegrity, 47 links, 46 joints
Links:
- removed link ball1
Joints:
- removed joint ball1

Commit message: added some comments on variables

File: data/tensegrity/robots/tensegrity.URDF (robot description, URDF)
Before this commit: robot tensegrity, 55 links, 54 joints
Joints:
- joint detach4: origin xyz=-0.15575 0.0165000000000074 1.57 rpy=1.5707963267949 0 3.14159265358979 -> xyz=-0.21575 0.0165000000000074 1.57 rpy=1.5707963267949 0 3.14159265358979
